File: ButtonGameController/Controller/Controller.kicad_pcb (KiCad board)
At the start: 2 copper layers, 85 x 43 mm, 34 parts, among them J1 FTDI Adapter, J2 2.4" Disp, Q1 AO3401A, Q2 AO3401A, Q3 AO3400A, SW1 BIG_BTN_SW (MH), SW2 BOOT, SW3 ON (MH), SW4 SW_SPST, U1 ESP32-WROOM-32, U2 ME6210A33PG

Commit message: screen config
Parts:
- removed BT1: 4xAAA (JST), Connector_PinHeader_2.54mm:PinHeader_1x02_P2.54mm_Vertical
- added BAT1: BAT, Connector_PinSocket_2.54mm:PinSocket_1x02_P2.54mm_Vertical, F.Cu at (105.0, 120.1)
- added C7: 10uF, Capacitor_SMD:C_0805_2012Metric, F.Cu at (118.2, 121.8)
- added C8: 10uF, Capacitor_SMD:C_0805_2012Metric, F.Cu at (118.2, 124.8)
- added D3: SMBJ6.5CA, custom-lib:D_SMB_Unidirectional, F.Cu at (111.8, 123.1)
- added J3: CHG_BREAKOUT, Connector_JST:JST_PH_B4B-PH-K_1x04_P2.00mm_Vertical, F.Cu at (127.9, 113.0)
- added J4: CHG, Connector_PinSocket_2.54mm:PinSocket_1x03_P2.54mm_Vertical, F.Cu at (122.6, 112.6)
- added Q4: AO3400A, Package_TO_SOT_SMD:SOT-23, F.Cu at (105.2, 111.2)
- added Q6: AO3400A, Package_TO_SOT_SMD:SOT-23, F.Cu at (105.2, 115.6)
- added R10: 5.1k, Resistor_SMD:R_0603_1608Metric, F.Cu at (100.7, 108.3)
- added R11: 5.1k, Resistor_SMD:R_0603_1608Metric, F.Cu at (100.7, 110.8)
- added R12: 1.2k, Resistor_SMD:R_0603_1608Metric, F.Cu at (100.7, 113.3)
- added R13: 5.1k, Resistor_SMD:R_0603_1608Metric, F.Cu at (100.7, 115.8)
- added R14: 5.1k, Resistor_SMD:R_0603_1608Metric, F.Cu at (100.7, 118.3)
- added R15: 5.1k, Resistor_SMD:R_0603_1608Metric, F.Cu at (100.7, 120.8)
- added R16: 1k, Resistor_SMD:R_0603_1608Metric, F.Cu at (126.9, 118.1)
- added R17: 1k, Resistor_SMD:R_0603_1608Metric, F.Cu at (126.9, 120.6)
- added R9: 5.1k, Resistor_SMD:R_0603_1608Metric, F.Cu at (100.7, 105.8)
- added U4: TP4056, Package_SO:SOIC-8-1EP_3.9x4.9mm_P1.27mm_EP2.41x3.3mm_ThermalVias, F.Cu at (111.8, 117.1)
- Q3: value AO3400A -> AO3401A; footprint SamacSys_Parts:SOT95P280X125-3N -> Package_TO_SOT_SMD:SOT-23
- moved Q3 39.1 mm to (105.2, 106.7), turned to 0 degrees
Connections:
- F1 pad 1: +BATT -> Net-(U4-CE)
- F1 pad 2: /HP_POSTFUSE -> +5V
- J1 pad 1: +BATT -> +5V
- Q2 pad 2: /HP_POSTFUSE -> +BATT
- Q3 pad 1: BTN_LED -> Net-(Q3-G)
- Q3 pad 2: GND -> +BATT
- Q3 pad 3: Net-(D1-K) -> Net-(Q3-D)
- R1 pad 1: /HP_POSTFUSE -> +BATT
- R8 pad 1: +3V8 -> +BATT
- U1 pad 33: unconnected-(U1-IO21-Pad33) -> BAT_IN
- U1 pad 36: unconnected-(U1-IO22-Pad36) -> BAT_EN
Routing:
- net +3V8: track 61.5 -> 0.00 mm, vias 2 -> 0
- net /HP_POSTFUSE: track 11.2 -> 0.00 mm
- net +BATT: track 10.5 -> 2.03 mm
- net Net-(D1-K): track 5.93 -> 0.00 mm
- net DISP_LED: track 57.8 -> 57.0 mm
- net T_CS: track 82.6 -> 82.1 mm
- net DBG: track 11.2 -> 10.6 mm
- net CS: track 75.9 -> 75.4 mm

Commit message: display calibration
Parts:
- removed G***2: LOGO, Graphics:logo_new
- added G***: LOGO, Graphics:logo_new_small, F.Cu at (122.8, 169.0)
- moved J4 59.4 mm to (101.6, 168.2), turned to -90 degrees
- moved R17 58.6 mm to (93.2, 168.6), turned to 180 degrees
- moved R16 55.0 mm to (105.0, 168.6)
- moved R9 53.2 mm to (94.4, 158.6)
- moved J3 52.4 mm to (97.0, 155.4), turned to 180 degrees
- moved R10 51.2 mm to (91.4, 158.6), turned to 180 degrees
- moved C7 46.6 mm to (101.6, 165.4), turned to 180 degrees
- moved D3 45.9 mm to (91.0, 164.0), turned to 90 degrees
- moved U4 44.1 mm to (104.8, 160.6), turned to -90 degrees
- moved R12 43.1 mm to (106.2, 156.0)
- moved BAT1 42.6 mm to (99.8, 162.5), turned to 180 degrees
- moved Q3 41.3 mm to (104.9, 148.0), turned to 90 degrees
- moved R11 40.2 mm to (104.9, 150.8), turned to 180 degrees
- moved Q4 37.1 mm to (100.8, 148.0), turned to 90 degrees
- moved R13 35.0 mm to (100.8, 150.8)
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Connections:
- net /MP_BB_G renamed /MP_BB_A
- net Net-(D1-K) renamed /MP_BB_C
- net Net-(U4-CE) renamed /HP_5V_FUSED
- R8 pad 1: +BATT -> +3V8
Routing:
- net BAT_EN: track 0.00 -> 66.5 mm, vias 0 -> 2
- net BAT_IN: track 0.00 -> 47.3 mm
- net +3V8: track 0.00 -> 45.3 mm, vias 0 -> 3
- net +BATT: track 2.03 -> 30.2 mm, vias 0 -> 2
- net /HP_5V_FUSED: track 0.00 -> 27.3 mm
- net +5V: track 0.00 -> 22.5 mm
- net Net-(U4-~{CHRG}): track 0.00 -> 21.3 mm
- net GND: track 3.90 -> 20.3 mm, vias 82 -> 83
- net MOSI: track 107.7 -> 116.3 mm
- net MISO: track 101.3 -> 109.8 mm
- net SCK: track 89.4 -> 97.8 mm
- net DC: track 77.6 -> 85.8 mm
- net Net-(U4-~{STDBY}): track 0.00 -> 6.22 mm
- net /MP_BB_C: track 0.00 -> 5.84 mm
- net Net-(Q3-G): track 0.00 -> 5.82 mm
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Other:
- board text added: "+"
- board text added: "C"
- board text added: "CHG"
- board text added: "PG"
- board text added: "SBY"
- board text added: "U+"
- board text added: "U-"
- board text removed: "!! REMOVE BATTERY BEFORE CONNECTING DEBUG !!"
- board text removed: "B+"
- board text removed: "PROG"
