File: ButtonGameController/Controller/Controller.kicad_sch (KiCad schematic)
At the start: 29 parts, among them J1 FTDI Adapter, J2 2.4" Disp, Q1 AO3401A, Q2 AO3401A, Q3 AO3400A, SW1 BIG_BTN_SW (MH), SW2 BOOT, SW3 ON (MH), SW4 SW_SPST, U1 ESP32-WROOM-32, U2 ME6210A33PG

Commit message: screen config
Parts:
- removed BT1: 4xAAA (JST), Connector_PinHeader_2.54mm:PinHeader_1x02_P2.54mm_Vertical, symbol Device:Battery
- removed Q3: AO3400A, SOT95P280X125-3N, symbol SamacSys_Parts:AO3400A
- added BAT1: BAT, Connector_PinSocket_2.54mm:PinSocket_1x02_P2.54mm_Vertical, symbol Connector:Conn_01x02_Male
- added C7, C8: 10uF, Capacitor_SMD:C_0805_2012Metric, symbol Device:C
- added D3: SMBJ6.5CA, custom-lib:D_SMB_Unidirectional, symbol Device:D_TVS
- added J3: CHG_BREAKOUT, Connector_JST:JST_PH_B4B-PH-K_1x04_P2.00mm_Vertical, symbol Connector:Conn_01x04_Socket
- added J4: CHG, Connector_PinSocket_2.54mm:PinSocket_1x03_P2.54mm_Vertical, symbol Connector:Conn_01x03_Socket
- added Q3: AO3401A, Package_TO_SOT_SMD:SOT-23, symbol Transistor_FET:AO3401A
- added Q4, Q6: AO3400A, Package_TO_SOT_SMD:SOT-23, symbol Transistor_FET:AO3400A
- added R10, R11, R13, R14, R15, R9: 5.1k, Resistor_SMD:R_0603_1608Metric, symbol Device:R
- added R12: 1.2k, Resistor_SMD:R_0603_1608Metric, symbol Device:R
- added R16, R17: 1k, Resistor_SMD:R_0603_1608Metric, symbol Device:R
- added U4: TP4056, Package_SO:SOIC-8-1EP_3.9x4.9mm_P1.27mm_EP2.41x3.3mm_ThermalVias, symbol Battery_Management:TP4056-42-ESOP8
Connections:
- net +3V8: no longer R8.1
- net +BATT: now also Q2.2 (S), R1.1, R8.1, BAT1.2 (Pin_2), C7.1, Q3.2 (S), R11.1, U4.5 (BAT); no longer F1.1, J1.1 (Pin_1)
- net BTN_LED: now also Q6.1 (G)
- net GND: now also BAT1.1 (Pin_1), C7.2, C8.2, D3.1 (A1), J3.1 (Pin_1), Q4.2 (S), Q6.2 (S), R10.2, R12.2, R13.2, R15.2, R9.2, U4.1 (TEMP), U4.3 (GND), U4.9 (EPAD)
- net at D1.1 (K): now also Q6.3 (D)
- net BAT_IN: now reaches U1.33 (IO21)
- net BAT_IN: now also R14.2, R15.1
- net BAT_EN: now reaches U1.36 (IO22)
- net BAT_EN: now also Q4.1 (G), R13.1
- removed net HP_POSTFUSE: F1.2, Q2.2 (S), R1.1
- new net: C8.1, F1.1, U4.4 (V_{CC}), U4.8 (CE)
- new net: R12.1, U4.2 (PROG)
- new net: R16.2, U4.6 (~{STDBY})
- new net: R17.2, U4.7 (~{CHRG})
- new net: J3.3 (Pin_3), R10.1
- new net: J3.2 (Pin_2), R9.1
- new net: Q3.1 (G), Q4.3 (D), R11.2
- new net: Q3.3 (D), R14.1
- new net +5V: D3.2 (A2), F1.2, J1.1 (Pin_1), J3.4 (Pin_4), J4.2 (Pin_2)
- new net CHRG: J4.1 (Pin_1), R16.1
- new net STDBY: J4.3 (Pin_3), R17.1
Other:
- note removed: "BAT IN"
- note removed: "REMOVE BAT BEFORE PLUGGING FTDI"
- moved on the sheet: D1, F1, R6, R7, R8, SW1

Commit message: display calibration
Connections:
- net +3V8: now also R8.1
- net +BATT: no longer R8.1
- net HP_5V_FUSED: now reaches C8.1, F1.1, U4.4 (V_{CC}), U4.8 (CE)
- net MP_BB_C: now reaches D1.1 (K), Q6.3 (D)
- net MP_BB_G renamed MP_BB_A
Changed lines of the file:
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@@
 		)
 	)
-	(label "MP_BB_G"
+	(label "HP_5V_FUSED"
+		(at 124.46 148.59 180)
+		(effects
+			(font
+				(size 1.27 1.27)
+			)
+			(justify right bottom)
+		)
+	)
+	(label "MP_BB_A"
 		(at 25.4 44.45 0)
 		(effects
@@
 		)
 	)
+	(label "MP_BB_C"
+		(at 25.4 60.96 0)
+		(effects
+			(font
+				(size 1.27 1.27)
+			)
+			(justify left bottom)
+		)
+	)
 	(global_label "CS"
 		(shape input)
@@
 	)
 	(symbol
+		(lib_id "power:+3V8")
+		(at 25.4 29.21 0)
+		(unit 1)
+		(body_style 1)
+		(exclude_from_sim no)
+		(in_bom yes)
+		(on_board yes)
+		(in_pos_files yes)
+		(dnp no)
+		(fields_autoplaced yes)
+		(property "Reference" "#PWR028"
+			(at 25.4 33.02 0)
+			(hide yes)
+			(show_name no)
+			(do_not_autoplace no)
+			(effects
+				(font
+					(size 1.27 1.27)
+				)
+			)
+		)
+		(property "Value" "+3V8"
+			(at 25.4 24.13 0)
+			(show_name no)
+			(do_not_autoplace no)
+			(effects
+				(font
+					(size 1.27 1.27)
+				)
+			)
+		)
+		(property "Footprint" ""
+			(at 25.4 29.21 0)
+			(hide yes)
+			(show_name no)
+			(do_not_autoplace no)
+			(effects
+				(font
+					(size 1.27 1.27)
+				)
+			)
+		)
+		(property "Datasheet" ""
+			(at 25.4 29.21 0)
+			(hide yes)
+			(show_name no)
+			(do_not_autoplace no)
+			(effects
+				(font
+					(size 1.27 1.27)
+				)
+			)
+		)
+		(property "Description" "Power symbol creates a global label with name \"+3V8\""
+			(at 25.4 29.21 0)
+			(hide yes)
+			(show_name no)
+			(do_not_autoplace no)
+			(effects
+				(font
+					(size 1.27 1.27)
+				)
+			)
+		)
+		(pin "1"
+		)
+		(instances
+			(project "Controller"
+				(path "/e6232cda-d5c6-423c-af59-e528087dcf2d"
+					(reference "#PWR028")
+					(unit 1)
+				)
+			)
+		)
+	)
+	(symbol
 		(lib_id "power:GND")
 		(at 250.19 67.31 0)
@@
 					(unit 1)
 				)
-			)
-		)
-	)
-	(symbol
-		(lib_id "power:+BATT")
-		(at 25.4 29.21 0)
-		(unit 1)
-		(body_style 1)
-		(exclude_from_sim no)
-		(in_bom yes)
-		(on_board yes)
-		(in_pos_files yes)
-		(dnp no)
-		(property "Reference" "#PWR037"
-			(at 25.4 33.02 0)
-			(hide yes)
-			(show_name no)
-			(do_not_autoplace no)
-			(effects
-				(font
-					(size 1.27 1.27)
-				)
-			)
-		)
-		(property "Value" "+BATT"
-			(at 25.781 24.8158 0)
-			(show_name no)
-			(do_not_autoplace no)
-			(effects
-				(font
-					(size 1.27 1.27)
-				)
-			)
-		)
-		(property "Footprint" ""
-			(at 25.4 29.21 0)
-			(hide yes)
-			(show_name no)
-			(do_not_autoplace no)
-			(effects
-				(font
-					(size 1.27 1.27)
-				)
-			)
-		)
-		(property "Datasheet" ""
-			(at 25.4 29.21 0)
-			(hide yes)
-			(show_name no)
-			(do_not_autoplace no)
-			(effects
-				(font
-					(size 1.27 1.27)
-				)
-			)
-		)
-		(property "Description" ""
-			(at 25.4 29.21 0)
-			(hide yes)
-			(show_name no)
-			(do_not_autoplace no)
-			(effects
-				(font
-					(size 1.27 1.27)
-				)
-			)
-		)
-		(pin "1"
-		)
-		(instances
-			(project "Controller"
-				(path "/e6232cda-d5c6-423c-af59-e528087dcf2d"
-					(reference "#PWR037")
-					(unit 1)
-				)
